Commit message: - added husky custom config - update husky control setting to coordinate with CMU navigation stack - add urdf for husky with different sensor configurations.. VLP16, D435i, Livox Mid360 - add urdf for a dummy custom platform that mount my custom platform on a husky - added husky_gazebo entry to use my custom husky - TODO: currenltly a bit messy in husky urdf file, need to fix hard-coded values to allow argument passing

File: husky_description/urdf/accessories/custom_platform_mount.urdf.xacro (robot description, xacro)
@@ -1,11 +1,8 @@
 <?xml version="1.0"?>
 <robot xmlns:xacro="http://wiki.ros.org/xacro">
-  <xacro:include filename="$(find velodyne_description)/urdf/VLP-16.urdf.xacro" />
-  <xacro:macro name="vlp16_mount" params="prefix parent_link topic height:=0.12 *origin">
-    <!--
-      The VLP16 is mounted to a pair of extrusion rods on top of the main sensor arch
-    -->
-    <link name="${prefix}vlp16_mount_base_link" />
-    <link name="${prefix}vlp16_mount_plate">
+  <xacro:include filename="$(find husky_description)/urdf/accessories/yadongliu_custom_platform.urdf.xacro"/>
+  <xacro:macro name="custom_platform_mount" params="prefix parent_link height:=0.12 *origin">
+    <link name="${prefix}platform_mount_base_link" />
+    <link name="${prefix}platform_mount_plate">
       <visual>
         <geometry>
@@ -24,5 +21,5 @@
       </collision>
     </link>
-    <link name="${prefix}vlp16_mount_left_support">
+    <link name="${prefix}platform_mount_left_support">
       <visual>
         <geometry>
@@ -41,5 +38,5 @@
       </collision>
     </link>
-    <link name="${prefix}vlp16_mount_right_support">
+    <link name="${prefix}platform_mount_right_support">
       <visual>
         <geometry>
@@ -58,27 +55,27 @@
       </collision>
     </link>
-    <joint name="${prefix}vlp16_mount_base_link_joint" type="fixed">
+    <joint name="${prefix}platform_mount_base_link_joint" type="fixed">
       <parent link="${parent_link}" />
-      <child link="${prefix}vlp16_mount_base_link" />
+      <child link="${prefix}platform_mount_base_link" />
       <xacro:insert_block name="origin" />
     </joint>
-    <joint name="${prefix}vlp16_mount_left_support_joint" type="fixed">
-      <parent link="${prefix}vlp16_mount_base_link" />
-      <child link="${prefix}vlp16_mount_left_support" />
+    <joint name="${prefix}platform_mount_left_support_joint" type="fixed">
+      <parent link="${prefix}platform_mount_base_link" />
+      <child link="${prefix}platform_mount_left_support" />
       <origin xyz="0 0.06 ${height/2}" rpy="0 0 0"/>
     </joint>
-    <joint name="${prefix}vlp16_mount_right_support_joint" type="fixed">
-      <parent link="${prefix}vlp16_mount_base_link" />
-      <child link="${prefix}vlp16_mount_right_support" />
+    <joint name="${prefix}platform_mount_right_support_joint" type="fixed">
+      <parent link="${prefix}platform_mount_base_link" />
+      <child link="${prefix}platform_mount_right_support" />
       <origin xyz="0 -0.06 ${height/2}" rpy="0 0 0"/>
     </joint>
-    <joint name="${prefix}vlp16_mount_plate_joint" type="fixed">
-      <parent link="${prefix}vlp16_mount_base_link" />
-      <child link="${prefix}vlp16_mount_plate" />
+    <joint name="${prefix}platform_mount_plate_joint" type="fixed">
+      <parent link="${prefix}platform_mount_base_link" />
+      <child link="${prefix}platform_mount_plate" />
       <origin xyz="0 0 ${height}" rpy="0 0 0"/>
     </joint>
-    <xacro:VLP-16 parent="${prefix}vlp16_mount_plate" topic="${topic}" name="${prefix}velodyne" hz="5" samples="350" min_range="0.01">
+    <!-- <xacro:VLP-16 parent="$_mount_plate" topic="${topic}" name="${prefix}velodyne" hz="5" samples="350" min_range="0.01">
       <origin xyz="0 0 0.0063" rpy="0 0 0" />
-    </xacro:VLP-16>
+    </xacro:VLP-16> -->
   </xacro:macro>
 </robot>

File: husky_description/urdf/husky.urdf.xacro (robot description, xacro)
@@ -23,6 +23,8 @@
 <robot name="husky" xmlns:xacro="http://ros.org/wiki/xacro">
   <!-- IMU Link -->
-  <xacro:arg name="imu_xyz"     default="$(optenv HUSKY_IMU_XYZ 0.19 0 0.149)"/>
-  <xacro:arg name="imu_rpy"     default="$(optenv HUSKY_IMU_RPY 0 -1.5708 3.1416)"/>
+  <!-- <xacro:arg name="imu_xyz"     default="$(optenv HUSKY_IMU_XYZ 0.19 0 0.149)"/>
+  <xacro:arg name="imu_rpy"     default="$(optenv HUSKY_IMU_RPY 0 -1.5708 3.1416)"/> -->
+  <xacro:arg name="imu_xyz"     default="$(optenv HUSKY_IMU_XYZ 0 0 0)"/>
+  <xacro:arg name="imu_rpy"     default="$(optenv HUSKY_IMU_RPY 0 0 0)"/>
   <xacro:arg name="imu_parent"  default="$(optenv HUSKY_IMU_PARENT base_link)"/>
   <!-- LMS1XX Laser Primary and Secondary -->
@@ -57,5 +59,6 @@
   <xacro:arg name="laser_3d_enabled"              default="$(optenv HUSKY_LASER_3D_ENABLED 0)" />
   <xacro:arg name="laser_3d_topic"                default="$(optenv HUSKY_LASER_3D_TOPIC points)"/>
-  <xacro:arg name="laser_3d_tower"                default="$(optenv HUSKY_LASER_3D_TOWER 1)"/>
+  <!-- NOTE: tmp -->
+  <xacro:arg name="laser_3d_tower"                default="$(optenv HUSKY_LASER_3D_TOWER 0)"/>
   <xacro:arg name="laser_3d_prefix"               default="$(optenv HUSKY_LASER_3D_PREFIX )"/>
   <xacro:arg name="laser_3d_parent"               default="$(optenv HUSKY_LASER_3D_PARENT top_plate_link)"/>
@@ -123,6 +126,12 @@
   <xacro:include filename="$(find husky_description)/urdf/accessories/sick_lms1xx_mount.urdf.xacro"/>
   <xacro:include filename="$(find husky_description)/urdf/accessories/vlp16_mount.urdf.xacro"/>
+  <xacro:include filename="$(find husky_description)/urdf/accessories/custom_platform_mount.urdf.xacro"/>
   <xacro:include filename="$(find husky_description)/urdf/decorations.urdf.xacro" />
   <xacro:include filename="$(find husky_description)/urdf/wheel.urdf.xacro" />
+  <!-- TODO: verify -->
+  <!-- <xacro:include filename="$(find husky_description)/urdf/accessories/yadongliu_custom_platform.urdf.xacro"/> -->
+  <xacro:custom_platform_mount prefix="$(arg laser_3d_prefix)" parent_link="$(arg laser_3d_parent)">
+    <origin xyz="$(arg laser_3d_xyz)" rpy="$(arg laser_3d_rpy)" />
+  </xacro:custom_platform_mount>
   <xacro:property name="M_PI" value="3.14159"/>
   <!-- Base Size -->
@@ -301,5 +310,5 @@
     </xacro:if>
     <xacro:unless value="$(arg laser_3d_tower)">
-      <xacro:VLP-16 parent="$(arg laser_3d_parent)" topic="$(arg laser_3d_topic)" name="$(arg laser_3d_prefix)velodyne">
+      <xacro:VLP-16 parent="$(arg laser_3d_parent)" topic="$(arg laser_3d_topic)" name="$(arg laser_3d_prefix)velodyne" hz="5" samples="350" min_range="0.01">
         <origin xyz="$(arg laser_3d_xyz)" rpy="$(arg laser_3d_rpy)" />
       </xacro:VLP-16>
